File: RO Flow Counter.sch (KiCad schematic (older format))
At the start: 29 parts, among them J7 Conn_01x02, J8 Conn_01x04, K1 G5Q-1A, Q1 BC807, Q2 BC807, Q3 2N7002E

Commit message: change to esp32
Connections:
- net mcu/TIM1_CH1 renamed mcu/FLOW_IN
Changed lines of the file:
@@
 F6 "RE_A" I L 5150 2725 50
 F7 "RE_B" I L 5150 2825 50
-F8 "TIM1_CH1" I L 5150 3125 50
-F9 "ERROR_OUT" O L 5150 5150 50
-F10 "LEVEL_IN" I L 5150 3225 50
-F11 "NORMAL_OPERATION_OUT" O L 5150 4550 50
-F12 "LCD_RS" O R 6675 4075 50
-F13 "RELAY_OUT" O R 6675 2650 50
-F14 "NRST" O R 6675 4175 50
-F15 "TIM3_CH2" O R 6675 4425 50
-F16 "TX" O R 6675 5625 50
-F17 "RX" I R 6675 5725 50
+F8 "ERROR_OUT" O L 5150 5150 50
+F9 "LEVEL_IN" I L 5150 3225 50
+F10 "NORMAL_OPERATION_OUT" O L 5150 4550 50
+F11 "LCD_RS" O R 6675 4075 50
+F12 "RELAY_OUT" O R 6675 2650 50
+F13 "NRST" O R 6675 4175 50
+F14 "TX" O R 6675 5625 50
+F15 "RX" I R 6675 5725 50
+F16 "FLOW_IN" I L 5150 3125 50
+F17 "LCD_BACKLIGHT" O R 6675 4425 50
 $EndSheet
 Wire Wire Line

Commit message: v1
Parts:
- removed TP10: LEVEL_OUT, TestPoint:TestPoint_Pad_D1.5mm, symbol Connector:TestPoint
- removed TP7: SPI_MOSI, TestPoint:TestPoint_Pad_D1.5mm, symbol Connector:TestPoint
- removed TP9: FLOW_OUT, TestPoint:TestPoint_Pad_D1.5mm, symbol Connector:TestPoint
- added R20: 1k, Resistor_SMD:R_0402_1005Metric, symbol Device:R
- J7: footprint Connector_Wire:SolderWire-0.25sqmm_1x02_P4.5mm_D0.65mm_OD2mm -> Connector_Wire:SolderWire-0.75sqmm_1x02_P7mm_D1.25mm_OD3.5mm
- TP11: value SPI_SCL1 -> SCL
- TP6: value SPI_CS -> SDA
- TP8: value LCD_RS -> RESET_LCD
Connections:
- net GND: now also R20.1
- net at Q3.1 (G), R7.1, TP4.1: now also R20.2
- net display/CS renamed display/SDA
- net display/RS renamed display/RESET_DISPLAY
Changed lines of the file:
@@
 F0 "display" 50
 F1 "../Filmant Dryer/display.sch" 50
-F2 "CS" I L 7400 3775 50
-F3 "SCL" I L 7400 3875 50
-F4 "MOSI" I L 7400 3975 50
-F5 "RS" I L 7400 4075 50
-F6 "NRST" I L 7400 4175 50
-F7 "BACKLIGHT_LCD" I L 7400 4425 50
+F2 "BACKLIGHT_LCD" I L 7400 4425 50
+F3 "RESET_DISPLAY" I L 7400 4075 50
+F4 "SCL" I L 7400 3875 50
+F5 "SDA" B L 7400 3775 50
 $EndSheet
-Wire Wire Line
-	6675 3975 7025 3975
 Wire Wire Line
 	7400 3875 6900 3875
@@
 F0 "mcu" 50
 F1 "../Filmant Dryer/mcu.sch" 50
-F2 "SPI1_CS" O R 6675 3775 50
-F3 "SPI1_SCL" O R 6675 3875 50
-F4 "SPI1_MOSI" O R 6675 3975 50
-F5 "SW_PRESS" I L 5150 2625 50
-F6 "RE_A" I L 5150 2725 50
-F7 "RE_B" I L 5150 2825 50
-F8 "ERROR_OUT" O L 5150 5150 50
-F9 "LEVEL_IN" I L 5150 3225 50
-F10 "NORMAL_OPERATION_OUT" O L 5150 4550 50
-F11 "LCD_RS" O R 6675 4075 50
-F12 "RELAY_OUT" O R 6675 2650 50
-F13 "NRST" O R 6675 4175 50
-F14 "TX" O R 6675 5625 50
-F15 "RX" I R 6675 5725 50
-F16 "FLOW_IN" I L 5150 3125 50
-F17 "LCD_BACKLIGHT" O R 6675 4425 50
+F2 "SW_PRESS" I L 5150 2625 50
+F3 "RE_A" I L 5150 2725 50
+F4 "RE_B" I L 5150 2825 50
+F5 "ERROR_OUT" O L 5150 5150 50
+F6 "LEVEL_IN" I L 5150 3225 50
+F7 "NORMAL_OPERATION_OUT" O L 5150 4550 50
+F8 "RELAY_OUT" O R 6675 2650 50
+F9 "TX" O R 6675 5625 50
+F10 "RX" I R 6675 5725 50
+F11 "FLOW_IN" I L 5150 3125 50
+F12 "LCD_BACKLIGHT" O R 6675 4425 50
+F13 "SCL" O R 6675 3875 50
+F14 "SDA" B R 6675 3775 50
+F15 "RESET_LCD" O R 6675 4075 50
 $EndSheet
 Wire Wire Line
@@
 	1    0    0    -1
 $EndComp
-Wire Wire Line
-	4375 3125 4550 3125
-Wire Wire Line
-	4375 3225 4900 3225
 $Comp
 L Relay:G5Q-1A K1
@@
 	1    0    0    -1
 $EndComp
-Wire Wire Line
-	8125 3125 8125 2975
-Wire Wire Line
-	7825 2650 7625 2650
 $Comp
 L Device:R R7
@@
 	7150 2650 6675 2650
 $Comp
-L power:GNDPWR #PWR027
-U 1 1 62E287F3
-P 8125 3125
-F 0 "#PWR027" H 8125 2925 50  0001 C CNN
-F 1 "GNDPWR" H 8129 2971 50  0000 C CNN
-F 2 "" H 8125 3075 50  0001 C CNN
-F 3 "" H 8125 3075 50  0001 C CNN
-	1    8125 3125
-	1    0    0    -1
-$EndComp
-$Comp
 L power:GNDPWR #PWR028
 U 1 1 62E29488
@@
 Wire Wire Line
 	8125 2975 8125 2850
-Wire Wire Line
-	6675 4175 7400 4175
 $Comp
 L Connector:TestPoint TP?
@@
 AR Path="/62D89C56/62E50F81" Ref="TP?"  Part="1"
 AR Path="/62E50F81" Ref="TP6"  Part="1"
-F 0 "TP6" H 6975 3050 50  0000 R CNN
-F 1 "SPI_CS" H 7100 3150 50  0000 R CNN
+F 0 "TP6" H 7000 3075 50  0000 R CNN
+F 1 "SDA" H 7000 3150 50  0000 R CNN
 F 2 "TestPoint:TestPoint_Pad_D1.5mm" H 7000 3000 50  0001 C CNN
 F 3 "~" H 7000 3000 50  0001 C CNN
@@
 AR Path="/62D89C56/62E5167F" Ref="TP?"  Part="1"
 AR Path="/62E5167F" Ref="TP11"  Part="1"
-F 0 "TP11" H 7275 3250 50  0000 R CNN
-F 1 "SPI_SCL1" H 7150 3325 50  0000 R CNN
+F 0 "TP11" H 7150 3250 50  0000 R CNN
+F 1 "SCL" H 7100 3325 50  0000 R CNN
 F 2 "TestPoint:TestPoint_Pad_D1.5mm" H 7100 3175 50  0001 C CNN
 F 3 "~" H 7100 3175 50  0001 C CNN
 	1    6900 3175
-	1    0    0    -1
-$EndComp
-$Comp
-L Connector:TestPoint TP?
-U 1 1 62E51A6D
-P 7025 3350
-AR Path="/62205316/62E51A6D" Ref="TP?"  Part="1"
-AR Path="/622422B2/62E51A6D" Ref="TP?"  Part="1"
-AR Path="/62D89C56/62E51A6D" Ref="TP?"  Part="1"
-AR Path="/62E51A6D" Ref="TP7"  Part="1"
-F 0 "TP7" H 7200 3400 50  0000 R CNN
-F 1 "SPI_MOSI" H 7425 3500 50  0000 R CNN
-F 2 "TestPoint:TestPoint_Pad_D1.5mm" H 7225 3350 50  0001 C CNN
-F 3 "~" H 7225 3350 50  0001 C CNN
-	1    7025 3350
 	1    0    0    -1
 $EndComp
@@
 AR Path="/62E52046" Ref="TP8"  Part="1"
 F 0 "TP8" H 7325 3600 50  0000 R CNN
-F 1 "LCD_RS" H 7475 3675 50  0000 R CNN
+F 1 "RESET_LCD" H 7600 3675 50  0000 R CNN
 F 2 "TestPoint:TestPoint_Pad_D1.5mm" H 7350 3550 50  0001 C CNN
 F 3 "~" H 7350 3550 50  0001 C CNN
@@
 Wire Wire Line
 	6900 3875 6675 3875
-Wire Wire Line
-	7025 3350 7025 3975
-Connection ~ 7025 3975
-Wire Wire Line
-	7025 3975 7400 3975
 Wire Wire Line
 	7150 3550 7150 4075
@@
 Wire Wire Line
 	4525 2625 5150 2625
-$Comp
-L Connector:TestPoint TP?
-U 1 1 62E6161B
-P 4550 3575
-AR Path="/62205316/62E6161B" Ref="TP?"  Part="1"
-AR Path="/622422B2/62E6161B" Ref="TP?"  Part="1"
-AR Path="/62D89C56/62E6161B" Ref="TP?"  Part="1"
-AR Path="/62E6161B" Ref="TP9"  Part="1"
-F 0 "TP9" H 4725 3625 50  0000 R CNN
-F 1 "FLOW_OUT" H 5025 3700 50  0000 R CNN
-F 2 "TestPoint:TestPoint_Pad_D1.5mm" H 4750 3575 50  0001 C CNN
-F 3 "~" H 4750 3575 50  0001 C CNN
-	1    4550 3575
-	-1   0    0    1
-$EndComp
-$Comp
-L Connector:TestPoint TP?
-U 1 1 62E639F1
-P 4900 3750
-AR Path="/62205316/62E639F1" Ref="TP?"  Part="1"
-AR Path="/622422B2/62E639F1" Ref="TP?"  Part="1"
-AR Path="/62D89C56/62E639F1" Ref="TP?"  Part="1"
-AR Path="/62E639F1" Ref="TP10"  Part="1"
-F 0 "TP10" H 5075 3800 50  0000 R CNN
-F 1 "LEVEL_OUT" H 5375 3875 50  0000 R CNN
-F 2 "TestPoint:TestPoint_Pad_D1.5mm" H 5100 3750 50  0001 C CNN
-F 3 "~" H 5100 3750 50  0001 C CNN
-	1    4900 3750
-	-1   0    0    1
-$EndComp
-Wire Wire Line
-	4900 3750 4900 3225
-Connection ~ 4900 3225
-Wire Wire Line
-	4900 3225 5150 3225
-Wire Wire Line
-	4550 3575 4550 3125
-Connection ~ 4550 3125
-Wire Wire Line
-	4550 3125 5150 3125
 $Comp
 L Device:Fuse F1
@@
 F 0 "J7" H 9205 2092 50  0000 L CNN
 F 1 "Conn_01x02" H 9205 2001 50  0000 L CNN
-F 2 "Connector_Wire:SolderWire-0.25sqmm_1x02_P4.5mm_D0.65mm_OD2mm" H 9125 2100 50  0001 C CNN
+F 2 "Connector_Wire:SolderWire-0.75sqmm_1x02_P7mm_D1.25mm_OD3.5mm" H 9125 2100 50  0001 C CNN
 F 3 "~" H 9125 2100 50  0001 C CNN
 	1    9125 2100
@@
 Wire Wire Line
 	6675 5725 7550 5725
+Wire Wire Line
+	4375 3225 5150 3225
+Wire Wire Line
+	4375 3125 5150 3125
+Wire Wire Line
+	7825 2650 7725 2650
+Wire Wire Line
+	8125 3350 8125 3225
+$Comp
+L power:GNDPWR #PWR027
+U 1 1 62E287F3
+P 8125 3350
+F 0 "#PWR027" H 8125 3150 50  0001 C CNN
+F 1 "GNDPWR" H 8129 3196 50  0000 C CNN
+F 2 "" H 8125 3300 50  0001 C CNN
+F 3 "" H 8125 3300 50  0001 C CNN
+	1    8125 3350
+	1    0    0    -1
+$EndComp
+$Comp
+L Device:R R20
+U 1 1 62ED8364
+P 7725 2925
+F 0 "R20" V 7518 2925 50  0000 C CNN
+F 1 "1k" V 7609 2925 50  0000 C CNN
+F 2 "Resistor_SMD:R_0402_1005Metric" V 7655 2925 50  0001 C CNN
+F 3 "~" H 7725 2925 50  0001 C CNN
+	1    7725 2925
+	-1   0    0    1
+$EndComp
+Connection ~ 8125 3225
+Wire Wire Line
+	8125 3225 8125 2975
+Wire Wire Line
+	7725 2775 7725 2650
+Connection ~ 7725 2650
+Wire Wire Line
+	7725 2650 7625 2650
+Wire Wire Line
+	7725 3075 7725 3225
+Wire Wire Line
+	7725 3225 8125 3225
 $EndSCHEMATC
