File: RO Flow Counter.kicad_pcb (KiCad board)
At the start: 2 copper layers, 100 x 55 mm, 80 parts, among them J1 LCD Power, J2 Conn_01x12, J3 Barrel_Jack, J5 Flow Meter, J6 Level Sensor (optional), J7 Conn_01x02, J8 Programming, K1 G5Q-1A, Q1 2N7002E, Q2 2N7002E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

Commit message: fix lcd pads
Parts:
- removed G***: LOGO, Custom Footprints:puppy_symbol
- J2: footprint Connector_PinSocket_1.27mm:PinSocket_1x12_P1.27mm_Vertical -> Connector_Pin:ERC1602
- moved J2 4.83 mm to (168.4, 102.3), turned to 180 degrees
- moved C3 1.92 mm to (153.7, 100.8)
- moved TP11 1.05 mm to (166.3, 101.9)
- moved TP8 0.90 mm to (171.6, 101.7)
Routing:
- net /display/RESET_DISPLAY: track 10.1 -> 12.2 mm
- net Net-(C3-Pad1): track 3.46 -> 2.48 mm
- net Net-(C3-Pad2): track 3.40 -> 2.46 mm
- net /display/SCL: track 30.9 -> 31.7 mm
